File: dwellness.sch (KiCad schematic (older format))
At the start: 12 parts

Commit message: Minimal changes to test diffing
Parts:
- J? (x5): symbol Connector:USB_OTG -> dwellness-rescue:USB_OTG-Connector
Other:
- moved on the sheet: D?
Changed lines of the file:
@@
 $EndDescr
 $Comp
-L Connector:USB_OTG J?
+L dwellness-rescue:USB_OTG-Connector J?
 U 1 1 61408180
 P 4050 5500
@@
 	2650 1750 3150 1750
 $Comp
-L Connector:USB_OTG J?
+L dwellness-rescue:USB_OTG-Connector J?
 U 1 1 6140725A
 P 2350 1850
@@
 L pspice:DIODE D?
 U 1 1 6148101E
-P 4550 4900
-F 0 "D?" V 4596 4772 50  0000 R CNN
-F 1 "DIODE" V 4505 4772 50  0000 R CNN
-F 2 "" H 4550 4900 50  0001 C CNN
-F 3 "~" H 4550 4900 50  0001 C CNN
-	1    4550 4900
+P 4600 4900
+F 0 "D?" V 4646 4772 50  0000 R CNN
+F 1 "DIODE" V 4555 4772 50  0000 R CNN
+F 2 "" H 4600 4900 50  0001 C CNN
+F 3 "~" H 4600 4900 50  0001 C CNN
+	1    4600 4900
 	1    0    0    -1
 $EndComp
@@
 	4050 2050 3750 2050
 $Comp
-L Connector:USB_OTG J?
+L dwellness-rescue:USB_OTG-Connector J?
 U 1 1 61405F9C
 P 8150 5100
@@
 $EndComp
 $Comp
-L Connector:USB_OTG J?
+L dwellness-rescue:USB_OTG-Connector J?
 U 1 1 61408F70
 P 6500 5500
@@
 	6900 5600 6900 5500
 $Comp
-L Connector:USB_OTG J?
+L dwellness-rescue:USB_OTG-Connector J?
 U 1 1 61401E9B
 P 8200 1850
@@
 	4050 2050 4050 5200
 Wire Wire Line
-	4250 4900 4350 4900
+	4250 4900 4400 4900
 Connection ~ 4250 4900
 Wire Wire Line
-	4750 4900 5200 4900
+	4800 4900 5200 4900
 Wire Wire Line
 	5200 4000 5200 4900
